File: Balloon Beacon.kicad_sch (KiCad schematic)
At the start: 51 parts, among them J1 PV Input, J2 Serial, J3 ICSP, J4 I2C, J6 GPS_ANT, Q1 AO3401A, U1 XC6206P332MR, U2 ATmega328PB-MU, U3 STC22K33048-26.000MT, U4 LM50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

Commit message: Last minute schematic changes....
Parts:
- removed U1: XC6206P332MR, Package_TO_SOT_SMD:SOT-23, symbol Regulator_Linear:APE8865N-24-HF-3
- added U1: CJ431, Package_TO_SOT_SMD:SOT-23, symbol Reference_Voltage:TL431DBZ
- C8: value 22 uF -> 0.1uF; footprint Capacitor_SMD:C_0603_1608Metric -> Capacitor_SMD:C_0402_1005Metric; JLCPCB C59461 -> C1525
- R6: value 1M -> 43k; JLCPCB C22935 -> C23172
- R7: value 1M -> 100k; footprint Resistor_SMD:R_0603_1608Metric -> Resistor_SMD:R_0402_1005Metric; JLCPCB C22935 -> C25741
Connections:
- net VDD is gone; now on net +3V3: C11.1, C16.1, C3.1, D1.1 (K), D2.1 (K), R6.1, U4.1 (VCC), U7.1 (K), U7.2 (REF)
- net +3V3: now also C13.1, JP1.2 (B), U6.8 (VCC), U6.9 (~{RESET}), U1.1 (K)
- net GND: now also U1.3 (A)
- net VDD_TST: now also U1.2 (REF)
Other:
- moved on the sheet: C11, C18, J3, U7, U8
